File: pcb/I2CMotorsForM5Stack.kicad_pcb (KiCad board)
At the start: 2 copper layers, 60 x 50 mm, 34 parts, among them J1 FFC_connector, J2 2x15socket, J3 Conn_01x06, J4 Conn_01x06, J5 Conn_01x04, U1 TB6612FNG, U2 ATmega328PB-MU

Commit message: Update revision to 2020.05
Other:
- board text added: "Rev2020.05"
- board text removed: "Rev2020.04"
Changed lines of the file:
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@@
     (effects (font (size 1 1) (thickness 0.15)))
   )
-  (gr_text Rev2020.04 (at 119.5488 98.5832) (layer B.SilkS)
+  (gr_text Rev2020.05 (at 119.5488 98.5832) (layer B.SilkS)
     (effects (font (size 1 1) (thickness 0.15)) (justify mirror))
   )
