File: pcb/I2cMotorsForM5Stack.sch (KiCad schematic (older format))
At the start: 26 parts, among them J1 FFC_connector, J2 2x15socket, J3 Conn_01x06, J4 Conn_01x06, J5 Conn_01x04, U1 TB6612FNG, U2 ATmega328PB-MU

Commit message: Update something
Parts:
- removed JP4: NO, Jumper:SolderJumper-2_P1.3mm_Open_RoundedPad1.0x1.5mm, symbol Device:Jumper_NO_Small
Connections:
- no-connect marks 2 -> 5
Changed lines of the file:
@@
 Wire Wire Line
 	5850 3600 6150 3600
-$Comp
-L Device:Jumper_NO_Small JP4
-U 1 1 5E6C43A4
-P 5750 3900
-F 0 "JP4" H 5750 4085 50  0000 C CNN
-F 1 "NO" H 5750 3994 50  0000 C CNN
-F 2 "Jumper:SolderJumper-2_P1.3mm_Open_RoundedPad1.0x1.5mm" H 5750 3900 50  0001 C CNN
-F 3 "~" H 5750 3900 50  0001 C CNN
-	1    5750 3900
-	1    0    0    -1
-$EndComp
-Wire Wire Line
-	5850 3900 5850 3700
-Wire Wire Line
-	5850 3700 6150 3700
-$Comp
-L power:+3V3 #PWR0122
-U 1 1 5E6C62E7
-P 5200 3900
-F 0 "#PWR0122" H 5200 3750 50  0001 C CNN
-F 1 "+3V3" H 5215 4073 50  0000 C CNN
-F 2 "" H 5200 3900 50  0001 C CNN
-F 3 "" H 5200 3900 50  0001 C CNN
-	1    5200 3900
-	1    0    0    -1
-$EndComp
-Wire Wire Line
-	5200 3900 5650 3900
 Wire Wire Line
 	2800 3250 2800 3650
@@
 	1    0    0    -1
 $EndComp
+NoConn ~ 6150 3900
+NoConn ~ 6150 3800
+NoConn ~ 6150 3700
 $EndSCHEMATC

Commit message: Separate HPWR to NC0-2 for Core2
Parts:
- removed JP3: NO, Jumper:SolderJumper-2_P1.3mm_Open_RoundedPad1.0x1.5mm, symbol Device:Jumper_NO_Small
Connections:
- removed net HPWR: J1.1 (Pin_1), J1.3 (Pin_3), J1.5 (Pin_5), J2.26 (Pin_26), J2.28 (Pin_28), J2.30 (Pin_30), J5.2 (Pin_2)
- new net NC0: J1.5 (Pin_5), J2.26 (Pin_26)
- new net NC1: J1.3 (Pin_3), J2.28 (Pin_28)
- new net NC2: J1.1 (Pin_1), J2.30 (Pin_30)
- no-connect marks 5 -> 7
Changed lines of the file:
@@
 Comment4 ""
 $EndDescr
-Wire Wire Line
-	10200 3000 10250 3000
-Wire Wire Line
-	10250 3000 10250 2900
-Wire Wire Line
-	10250 2800 10200 2800
-Wire Wire Line
-	10200 2900 10250 2900
-Connection ~ 10250 2900
-Wire Wire Line
-	10250 2900 10250 2800
 $Comp
 L power:GND #PWR0109
@@
 Wire Wire Line
 	10350 1700 10350 1800
-Text Label 10250 3000 0    50   ~ 0
-HPWR
 Text Label 10200 2700 0    50   ~ 0
 15
@@
 	1    0    0    -1
 $EndComp
-$Comp
-L Device:Jumper_NO_Small JP3
-U 1 1 5E6C124E
-P 5750 3600
-F 0 "JP3" H 5750 3785 50  0000 C CNN
-F 1 "NO" H 5750 3694 50  0000 C CNN
-F 2 "Jumper:SolderJumper-2_P1.3mm_Open_RoundedPad1.0x1.5mm" H 5750 3600 50  0001 C CNN
-F 3 "~" H 5750 3600 50  0001 C CNN
-	1    5750 3600
-	1    0    0    -1
-$EndComp
-$Comp
-L power:GND #PWR0121
-U 1 1 5E6C1999
-P 5450 3600
-F 0 "#PWR0121" H 5450 3350 50  0001 C CNN
-F 1 "GND" H 5455 3427 50  0000 C CNN
-F 2 "" H 5450 3600 50  0001 C CNN
-F 3 "" H 5450 3600 50  0001 C CNN
-	1    5450 3600
-	1    0    0    -1
-$EndComp
-Wire Wire Line
-	5450 3600 5650 3600
-Wire Wire Line
-	5850 3600 6150 3600
 Wire Wire Line
 	2800 3250 2800 3650
@@
 Connection ~ 9700 2100
 Connection ~ 10200 1600
-Connection ~ 10200 2800
 Connection ~ 9700 2900
-Connection ~ 10200 2900
 Connection ~ 9700 3000
-Connection ~ 10200 3000
 Connection ~ 10200 1700
 Connection ~ 10200 1800
@@
 	1    0    0    -1
 $EndComp
-Text Label 5000 5400 0    50   ~ 0
-HPWR
 Wire Wire Line
 	5200 5300 5000 5300
+$Comp
+L power:+BATT #PWR0124
+U 1 1 5EAFD8AA
+P 5200 5300
+F 0 "#PWR0124" H 5200 5150 50  0001 C CNN
+F 1 "+BATT" H 5215 5473 50  0000 C CNN
+F 2 "" H 5200 5300 50  0001 C CNN
+F 3 "" H 5200 5300 50  0001 C CNN
+	1    5200 5300
+	1    0    0    -1
+$EndComp
+NoConn ~ 6150 3900
+NoConn ~ 6150 3800
+NoConn ~ 6150 3700
+Text Label 10200 2800 0    50   ~ 0
+NC0
+Text Label 10200 2900 0    50   ~ 0
+NC1
+Text Label 10200 3000 0    50   ~ 0
+NC2
+NoConn ~ 6150 3600
+Wire Wire Line
+	5000 5500 5400 5500
+NoConn ~ 5000 5400
 $Comp
 L power:+3V3 #PWR0123
@@
 	1    0    0    -1
 $EndComp
-Wire Wire Line
-	5000 5500 5400 5500
-$Comp
-L power:+BATT #PWR0124
-U 1 1 5EAFD8AA
-P 5200 5300
-F 0 "#PWR0124" H 5200 5150 50  0001 C CNN
-F 1 "+BATT" H 5215 5473 50  0000 C CNN
-F 2 "" H 5200 5300 50  0001 C CNN
-F 3 "" H 5200 5300 50  0001 C CNN
-	1    5200 5300
-	1    0    0    -1
-$EndComp
-NoConn ~ 6150 3900
-NoConn ~ 6150 3800
-NoConn ~ 6150 3700
 $EndSCHEMATC

Commit message: Update pdf of schematic
Parts:
- ADDR0, ADDR2, ADDR3, ADDR5, ADDR7, JP2: symbol Device:Jumper_NO_Small -> I2cMotorsForM5Stack-rescue:Jumper_NO_Small-Device
- ADDR1, ADDR4, ADDR6, JP1: symbol Device:Jumper_NC_Small -> I2cMotorsForM5Stack-rescue:Jumper_NC_Small-Device
- U1: symbol Driver_Motor:TB6612FNG -> I2cMotorsForM5Stack-rescue:TB6612FNG-Driver_Motor
- U2: symbol MCU_Microchip_ATmega:ATmega328PB-MU -> I2cMotorsForM5Stack-rescue:ATmega328PB-MU-MCU_Microchip_ATmega
Changed lines of the file:
@@
 RST
 $Comp
-L Driver_Motor:TB6612FNG U1
+L I2cMotorsForM5Stack-rescue:TB6612FNG-Driver_Motor U1
 U 1 1 5E409F59
 P 2500 5100
@@
 $EndComp
 $Comp
-L Device:Jumper_NC_Small JP1
+L I2cMotorsForM5Stack-rescue:Jumper_NC_Small-Device JP1
 U 1 1 5E41A7F4
 P 7950 3250
@@
 $EndComp
 $Comp
-L Device:Jumper_NO_Small JP2
+L I2cMotorsForM5Stack-rescue:Jumper_NO_Small-Device JP2
 U 1 1 5E41CE9B
 P 8250 3250
@@
 $EndComp
 $Comp
-L MCU_Microchip_ATmega:ATmega328PB-MU U2
+L I2cMotorsForM5Stack-rescue:ATmega328PB-MU-MCU_Microchip_ATmega U2
 U 1 1 5E68D65A
 P 6750 3100
@@
 $EndComp
 $Comp
-L Device:Jumper_NC_Small ADDR1
+L I2cMotorsForM5Stack-rescue:Jumper_NC_Small-Device ADDR1
 U 1 1 5E84FB49
 P 2350 2000
@@
 $EndComp
 $Comp
-L Device:Jumper_NO_Small ADDR0
+L I2cMotorsForM5Stack-rescue:Jumper_NO_Small-Device ADDR0
 U 1 1 5E8501F7
 P 2350 1900
@@
 	2000 1900 2000 2000
 $Comp
-L Device:Jumper_NO_Small ADDR2
+L I2cMotorsForM5Stack-rescue:Jumper_NO_Small-Device ADDR2
 U 1 1 5E855E5F
 P 2350 2100
@@
 $EndComp
 $Comp
-L Device:Jumper_NO_Small ADDR3
+L I2cMotorsForM5Stack-rescue:Jumper_NO_Small-Device ADDR3
 U 1 1 5E855FAF
 P 2350 2200
@@
 $EndComp
 $Comp
-L Device:Jumper_NC_Small ADDR4
+L I2cMotorsForM5Stack-rescue:Jumper_NC_Small-Device ADDR4
 U 1 1 5E8560B1
 P 2350 2300
@@
 $EndComp
 $Comp
-L Device:Jumper_NO_Small ADDR5
+L I2cMotorsForM5Stack-rescue:Jumper_NO_Small-Device ADDR5
 U 1 1 5E856295
 P 2350 2400
@@
 $EndComp
 $Comp
-L Device:Jumper_NC_Small ADDR6
+L I2cMotorsForM5Stack-rescue:Jumper_NC_Small-Device ADDR6
 U 1 1 5E856411
 P 2350 2500
@@
 $EndComp
 $Comp
-L Device:Jumper_NO_Small ADDR7
+L I2cMotorsForM5Stack-rescue:Jumper_NO_Small-Device ADDR7
 U 1 1 5E8565AF
 P 2350 2600
